File: Board_Schematics/Sensors_to_mcu_v0.1.sch (EAGLE design)
At the start: 37 parts, among them IC10 74AHC1G08DBV, IC11 74AHC1G08DBV, IC12 74AHC1G08DBV, IC13 74AHC1G08DBV, IC14 74AHC1G08DBV, IC15 74AHC1G08DBV, IC16 74AHC1G08DBV, IC17 74AHC1G08DBV, IC7 4022N, X1 INVERTER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

Commit message: Sensor measurement update
Added sensor signal
Parts:
- added ESP_VOLTAGE: PIN1-2, con-faston:PIN1-2
- added R1: (no value), rcl:R-EU_0207/10
- added SENSOR: (no value), rcl:C-EU025-025X050
- added SENSOR_MEASUREMENT: SV_ X, con-faston:PIN1-2
- added T1: BC547, transistor:BC547
- renumbered SV14 to ESP_PIN3, SV23 to ESP_PIN4, SV8 to ESP_PIN1, SV9 to ESP_PIN2
Connections:
- new net N$1: R1.1, SENSOR.1
- new net N$2: SENSOR.2, T1.B
- new net N$3: SENSOR_MEASUREMENT.1, T1.E
- new net N$4: ESP_VOLTAGE.1, R1.2
- new net VCC: T1.C
